Commit message: Added new URDF, some helpers

File: model/werdna_stand_bullet.urdf (robot description, URDF)
Before this commit: robot werdna, 8 links, 7 joints
Links:
- link base_link: mass 4.0 -> 3.0
- link left_wheel: geometry collision sphere radius=0.0855; visual cylinder length=0.045 radius=0.0855
- link right_wheel: geometry collision sphere radius=0.0855; visual cylinder length=0.045 radius=0.0855
Joints:
- joint left_hip_joint: origin xyz=0.0 0.1 0.0 rpy=0.0 1.571 0.0 -> xyz=0.0 0.1 0.0 rpy=0.0 1.318116071652818 0.0
- joint left_knee_joint: origin xyz=0.0 0.05 -0.2 rpy=0.0 0.0 0.0 -> xyz=0.0 0.05 -0.2 rpy=0.0 0.5053605102841575 0.0
- joint right_hip_joint: origin xyz=0.0 -0.1 0.0 rpy=0.0 1.571 0.0 -> xyz=0.0 -0.1 0.0 rpy=0.0 1.318116071652818 0.0
- joint right_knee_joint: origin xyz=0.0 -0.05 -0.2 rpy=0.0 0.0 0.0 -> xyz=0.0 -0.05 -0.2 rpy=0.0 0.5053605102841575 0.0

Commit message: Trained Agent

File: model/werdna_stand_bullet.urdf (robot description, URDF)
Before this commit: robot werdna, 8 links, 7 joints
Links:
- link left_wheel: geometry collision cylinder length=0.045 radius=0.0885; visual cylinder length=0.045 radius=0.0855
- link right_wheel: geometry collision cylinder length=0.045 radius=0.0885; visual cylinder length=0.045 radius=0.0855
